File: pcb/monkeyboard/monkeyboard.kicad_sch (KiCad schematic)
At the start: 152 parts

Commit message: u
Parts:
- Backspace1: renamed from Backspace; footprint Button_Switch_Keyboard:SW_Cherry_MX_1.00u_PCB -> Button_Switch_Keyboard:SW_Cherry_MX_2.00u_PCB
- Caps1: renamed from Caps; footprint Button_Switch_Keyboard:SW_Cherry_MX_1.00u_PCB -> Button_Switch_Keyboard:SW_Cherry_MX_1.75u_PCB
- Enter1: renamed from Enter; footprint Button_Switch_Keyboard:SW_Cherry_MX_1.00u_PCB -> Button_Switch_Keyboard:SW_Cherry_MX_2.25u_PCB
- Fn1: renamed from Fn; footprint Button_Switch_Keyboard:SW_Cherry_MX_1.00u_PCB -> Button_Switch_Keyboard:SW_Cherry_MX_1.25u_PCB
- LAlt1: renamed from LAlt; footprint Button_Switch_Keyboard:SW_Cherry_MX_1.00u_PCB -> Button_Switch_Keyboard:SW_Cherry_MX_1.25u_PCB
- LCtrl1: renamed from LCtrl; footprint Button_Switch_Keyboard:SW_Cherry_MX_1.00u_PCB -> Button_Switch_Keyboard:SW_Cherry_MX_1.25u_PCB
- LShift1: renamed from LShift; footprint Button_Switch_Keyboard:SW_Cherry_MX_1.00u_PCB -> Button_Switch_Keyboard:SW_Cherry_MX_2.25u_PCB
- Menu1: renamed from Menu; footprint Button_Switch_Keyboard:SW_Cherry_MX_1.00u_PCB -> Button_Switch_Keyboard:SW_Cherry_MX_1.25u_PCB
- Numpad0: footprint Button_Switch_Keyboard:SW_Cherry_MX_1.00u_PCB -> Button_Switch_Keyboard:SW_Cherry_MX_2.00u_PCB
- RAlt1: renamed from RAlt; footprint Button_Switch_Keyboard:SW_Cherry_MX_1.00u_PCB -> Button_Switch_Keyboard:SW_Cherry_MX_1.25u_PCB
- RCtrl1: renamed from RCtrl; footprint Button_Switch_Keyboard:SW_Cherry_MX_1.00u_PCB -> Button_Switch_Keyboard:SW_Cherry_MX_1.25u_PCB
- RShift1: renamed from RShift; footprint Button_Switch_Keyboard:SW_Cherry_MX_1.00u_PCB -> Button_Switch_Keyboard:SW_Cherry_MX_2.75u_PCB
- Space1: renamed from Space; footprint Button_Switch_Keyboard:SW_Cherry_MX_1.00u_PCB -> Button_Switch_Keyboard:SW_Cherry_MX_6.25u_PCB
- Tab1: renamed from Tab; footprint Button_Switch_Keyboard:SW_Cherry_MX_1.00u_PCB -> Button_Switch_Keyboard:SW_Cherry_MX_1.50u_PCB
- Win1: renamed from Win; footprint Button_Switch_Keyboard:SW_Cherry_MX_1.00u_PCB -> Button_Switch_Keyboard:SW_Cherry_MX_1.25u_PCB
- \1: renamed from \; footprint Button_Switch_Keyboard:SW_Cherry_MX_1.00u_PCB -> Button_Switch_Keyboard:SW_Cherry_MX_1.50u_PCB
- gave numbers to parts that had none: 76
- renumbered ' to '1, , to ,1, - to -1, . to .1, / to /1, ; to ;1, = to =1, A to A1, B to B1, C to C1, D to D21, Del to Del1, Down to Down1, E to E1, End to End1, F to F1, G to G1, H to H1, Home to Home1, I to I1, Ins to Ins1, J to J1, K to K1, L to L1, Left to Left1, M to M1, N to N1, O to O1, P to P1, PgDn to PgDn1, PgUp to PgUp1, Q to Q1, R to R1, Right to Right1, S to S1, T to T1, U to U1, Up to Up1, V to V1, W to W1, X to X1, Y to Y1, Z to Z1, [ to [1, ] to ]1, ` to `1
Connections:
- net C9: now also .1.2 (B), L1.2 (B), Num9.2 (B), O1.2 (B)
